File: PCB/AFF314KEEB.kicad_pcb (KiCad board)
At the start: 2 copper layers, 251.7 x 104.3 mm, 87 parts, among them SW1 RotaryEncoder_Switch, U1 Nice_Nano_V2

Commit message: Update
Parts:
- U1: moved to F.Cu
- turned U1 to 0 degrees
Connections:
- U1 pad 10: COL_3 -> COL_7
- U1 pad 11: COL_4 -> COL_6
- U1 pad 12: ROW_3 -> COL_5
- U1 pad 13: COL_5 -> A
- U1 pad 14: COL_6 -> B
- U1 pad 15: COL_7 -> ROW_3
- U1 pad 16: COL_8 -> COL_4
- U1 pad 17: COL_9 -> COL_3
- U1 pad 18: ROW_2 -> COL_2
- U1 pad 19: ROW_1 -> COL_1
- U1 pad 20: ROW_0 -> COL_0
- U1 pad 5: A -> ROW_0
- U1 pad 6: B -> ROW_1
- U1 pad 7: COL_0 -> ROW_2
- U1 pad 8: COL_1 -> COL_9
- U1 pad 9: COL_2 -> COL_8
Routing:
- net GND: track 113.0 -> 71.6 mm
- net ROW_3: track 182.9 -> 204.5 mm
- net A: track 47.7 -> 27.8 mm
- net B: track 50.0 -> 32.4 mm
- net BAT+: track 26.0 -> 10.7 mm
- net RESET: track 16.8 -> 25.3 mm
- net COL_4: track 188.6 -> 186.4 mm
- net COL_3: track 196.0 -> 193.8 mm
- net COL_2: track 224.5 -> 222.3 mm
- net COL_0: track 210.1 -> 207.8 mm
- net COL_6: track 201.3 -> 203.4 mm
- net COL_9: track 210.5 -> 212.4 mm
- net VBAT: track 50.4 -> 49.2 mm
- net ROW_0: track 259.5 -> 258.6 mm

Commit message: Small PCB tweak
Parts:
- moved DL37 1.48 mm to (157.4, 109.5)
Routing:
- net ROW_3: track 204.5 -> 196.3 mm
- net SW37_2: track 11.1 -> 12.5 mm
- net ROW_2: track 259.5 -> 260.3 mm
Changed lines of the file:
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@@
 			)
 		)
+		(model "${KIPRJMOD}/AFFE3D/AFF314KEEB_case.step"
+			(offset
+				(xyz -150 78 -4.5)
+			)
+			(scale
+				(xyz 1 1 1)
+			)
+			(rotate
+				(xyz -0 -0 -0)
+			)
+		)
 	)
 	(footprint "MountingHole:MountingHole_2.2mm_M2_DIN965_Pad_TopBottom"
@@
 		(placed yes)
 		(layer "B.Cu")
-		(at 155.91 109.66 90)
+		(at 157.38 109.5 90)
 		(descr "Diode, DO-41, SOD81, Horizontal, RM 10mm,")
 		(tags "Diode, DO-41, SOD81, Horizontal, RM 10mm, 1N4007, SB140,")
@@
 	)
 	(segment
-		(start 155.637111 78.824463)
-		(end 157.302065 78.824463)
-		(width 0.2)
-		(layer "B.Cu")
-		(net 24)
-	)
-	(segment
 		(start 231.822735 91.848601)
 		(end 231.822735 91.087031)
@@
 	)
 	(segment
-		(start 56.592425 95.345316)
-		(end 60.887329 91.050412)
+		(start 192.597811 106.968985)
+		(end 185.446587 106.968985)
 		(width 0.2)
 		(layer "B.Cu")
@@
 	)
 	(segment
-		(start 250.236892 90.745805)
-		(end 258.700228 99.209141)
+		(start 56.592425 95.345316)
+		(end 60.887329 91.050412)
 		(width 0.2)
 		(layer "B.Cu")
@@
 	)
 	(segment
-		(start 197.133708 102.433088)
-		(end 192.597811 106.968985)
+		(start 197.133708 101.671518)
+		(end 197.133708 102.433088)
 		(width 0.2)
 		(layer "B.Cu")
@@
 	)
 	(segment
-		(start 113.886218 103.80474)
-		(end 131.632142 103.80474)
+		(start 250.236892 90.745805)
+		(end 258.700228 99.209141)
 		(width 0.2)
 		(layer "B.Cu")
@@
 	)
 	(segment
-		(start 148.504765 86.932117)
-		(end 148.504765 85.956809)
+		(start 197.133708 102.433088)
+		(end 192.597811 106.968985)
 		(width 0.2)
 		(layer "B.Cu")
@@
 	)
 	(segment
+		(start 141.574411 80.001763)
+		(end 156.124765 80.001763)
+		(width 0.2)
+		(layer "B.Cu")
+		(net 24)
+	)
+	(segment
+		(start 185.446587 106.968985)
+		(end 157.302065 78.824463)
+		(width 0.2)
+		(layer "B.Cu")
+		(net 24)
+	)
+	(segment
 		(start 197.925258 102.463068)
 		(end 209.873239 102.463068)
@@
 	)
 	(segment
-		(start 158.880365 79.123893)
-		(end 158.880365 78.824463)
+		(start 113.886218 103.80474)
+		(end 117.771434 103.80474)
 		(width 0.2)
 		(layer "B.Cu")
@@
 	)
 	(segment
-		(start 148.504765 85.956809)
-		(end 155.637111 78.824463)
+		(start 156.124765 80.001763)
+		(end 157.302065 78.824463)
 		(width 0.2)
 		(layer "B.Cu")
@@
 	)
 	(segment
-		(start 131.632142 103.80474)
-		(end 148.504765 86.932117)
-		(width 0.2)
-		(layer "B.Cu")
-		(net 24)
-	)
-	(segment
 		(start 79.197191 94.408618)
 		(end 87.335815 102.547242)
@@
 	)
 	(segment
-		(start 186.725457 106.968985)
-		(end 158.880365 79.123893)
-		(width 0.2)
-		(layer "B.Cu")
-		(net 24)
-	)
-	(segment
 		(start 110.737799 106.953159)
 		(end 113.886218 103.80474)
@@
 	)
 	(segment
-		(start 192.597811 106.968985)
-		(end 186.725457 106.968985)
+		(start 197.133708 101.671518)
+		(end 197.925258 102.463068)
 		(width 0.2)
 		(layer "B.Cu")
@@
 	)
 	(segment
-		(start 197.133708 101.671518)
-		(end 197.925258 102.463068)
+		(start 117.771434 103.80474)
+		(end 141.574411 80.001763)
 		(width 0.2)
 		(layer "B.Cu")
@@
 	)
 	(segment
-		(start 197.133708 101.671518)
-		(end 197.133708 102.433088)
-		(width 0.2)
-		(layer "B.Cu")
-		(net 24)
-	)
-	(segment
 		(start 87.335815 102.547242)
 		(end 93.237002 102.547242)
@@
 	)
 	(segment
+		(start 171.084215 138.381149)
+		(end 165.48 132.776934)
+		(width 0.2)
+		(layer "B.Cu")
+		(net 25)
+	)
+	(segment
 		(start 189.470583 139.027363)
 		(end 176.182966 139.027363)
@@
 	)
 	(segment
-		(start 175.536752 138.381149)
-		(end 171.084215 138.381149)
+		(start 157.38 111.72)
+		(end 157.38 111.2)
 		(width 0.2)
 		(layer "B.Cu")
@@
 	)
 	(segment
-		(start 163.156071 130.453005)
-		(end 163.156071 118.606071)
+		(start 130.654831 128.702409)
+		(end 130.654831 97.851697)
 		(width 0.2)
 		(layer "B.Cu")
@@
 	)
 	(segment
-		(start 158.479365 108.790635)
-		(end 158.479365 78.336809)
+		(start 165.48 132.776934)
+		(end 165.48 119.82)
 		(width 0.2)
 		(layer "B.Cu")
@@
 	)
 	(segment
-		(start 141.14424 118.213)
-		(end 152.74031 118.213)
+		(start 145.73 100.21)
+		(end 147.86 98.08)
 		(width 0.2)
 		(layer "B.Cu")
@@
 	)
 	(segment
-		(start 130.654831 128.702409)
-		(end 141.14424 118.213)
+		(start 147.86 92.242398)
+		(end 142.062065 86.444463)
 		(width 0.2)
 		(layer "B.Cu")
@@
 	)
 	(segment
-		(start 200.009247 128.488699)
-		(end 189.470583 139.027363)
+		(start 145.73 101.98331)
+		(end 145.73 100.21)
 		(width 0.2)
 		(layer "B.Cu")
@@
 	)
 	(segment
-		(start 108.725248 131.778357)
-		(end 109.832915 130.67069)
+		(start 200.009247 128.488699)
+		(end 189.470583 139.027363)
 		(width 0.2)
 		(layer "B.Cu")
@@
 	)
 	(segment
-		(start 156.814411 77.647163)
-		(end 156.038111 78.423463)
+		(start 147.86 98.08)
+		(end 147.86 92.242398)
 		(width 0.2)
 		(layer "B.Cu")
@@
 	)
 	(segment
-		(start 157.789719 77.647163)
-		(end 156.814411 77.647163)
+		(start 108.725248 131.778357)
+		(end 109.832915 130.67069)
 		(width 0.2)
 		(layer "B.Cu")
@@
 	)
 	(segment
-		(start 200.009247 125.143674)
-		(end 213.430119 125.143674)
+		(start 157.38 111.2)
+		(end 154.94669 111.2)
 		(width 0.2)
 		(layer "B.Cu")
@@
 	)
 	(segment
-		(start 171.084215 138.381149)
-		(end 163.156071 130.453005)
+		(start 154.94669 111.2)
+		(end 145.73 101.98331)
 		(width 0.2)
 		(layer "B.Cu")
@@
 	)
 	(segment
-		(start 155.91 115.04331)
-		(end 155.91 111.36)
+		(start 200.009247 125.143674)
+		(end 213.430119 125.143674)
 		(width 0.2)
 		(layer "B.Cu")
@@
 	)
 	(segment
-		(start 152.74031 118.213)
-		(end 155.91 115.04331)
+		(start 165.48 119.82)
+		(end 157.38 111.72)
 		(width 0.2)
 		(layer "B.Cu")
@@
 	)
 	(segment
-		(start 155.91 111.36)
-		(end 158.479365 108.790635)
+		(start 130.654831 97.851697)
+		(end 142.062065 86.444463)
 		(width 0.2)
 		(layer "B.Cu")
@@
 	)
 	(segment
-		(start 156.038111 78.423463)
-		(end 150.083065 78.423463)
-		(width 0.2)
-		(layer "B.Cu")
-		(net 25)
-	)
-	(segment
-		(start 158.479365 78.336809)
-		(end 157.789719 77.647163)
+		(start 175.536752 138.381149)
+		(end 171.084215 138.381149)
 		(width 0.2)
 		(layer "B.Cu")
@@
 	)
 	(segment
-		(start 150.083065 78.423463)
-		(end 142.062065 86.444463)
-		(width 0.2)
-		(layer "B.Cu")
-		(net 25)
-	)
-	(segment
-		(start 163.156071 118.606071)
-		(end 155.91 111.36)
-		(width 0.2)
-		(layer "B.Cu")
-		(net 25)
-	)
-	(segment
 		(start 87.58291 119.600138)
 		(end 81.759554 119.600138)
@@
 	)
 	(segment
-		(start 153.21 107.96)
+		(start 153.05 107.8)
 		(end 147.3 102.05)
 		(width 0.2)
@@
 	)
 	(segment
-		(start 155.91 107.96)
-		(end 153.21 107.96)
+		(start 157.38 107.8)
+		(end 153.05 107.8)
 		(width 0.2)
 		(layer "B.Cu")

Commit message: Update
Parts:
- moved DL37 8.93 mm to (150.0, 104.5), turned to 0 degrees
Routing:
- net SW37_2: track 12.5 -> 5.40 mm
- net ROW_3: track 196.3 -> 194.8 mm
